Commit message: Neck component properly configured.

File: urdf/neck.urdf.xacro (robot description, xacro)
@@ -8,8 +8,23 @@
   <xacro:include filename="$(find schunk_description)/urdf/pw70/pw70.urdf.xacro" />
   <!-- Used for fixing robot to Gazebo -->
-  <link name="world"/>
-  <!-- arm -->
-  <xacro:schunk_pw70 name="neck" parent="world" >
-    <origin xyz="0 0 0" rpy="0 0 0" />
+  <!-- <link name="world"/> -->
+  <!-- neck -->
+  <link name="base_link">
+  <xacro:default_inertial/>
+  <!--
+  <visual>
+     <geometry>
+        <mesh filename="package://schunk_description/meshes/pw70/pw70_base.dae" />
+     </geometry>
+  </visual>
+  <collision>
+     <geometry>
+        <mesh filename="package://schunk_description/meshes/pw70/pw70_base.stl" />
+     </geometry>
+  </collision>
+          -->
+  </link>
+  <xacro:schunk_pw70 name="neck" parent="base_link" >
+    <origin xyz="0 -0.24 0.836" rpy="0 0 ${-1/2 * M_PI}" />
   </xacro:schunk_pw70>
   <!-- gazebo_plugin for arm -->
