Commit message: Addded new launch files

File: urdf/raw3-5.urdf.xacro (robot description, xacro)
@@ -8,4 +8,5 @@
   <xacro:include filename="$(find schunk_description)/urdf/materials.urdf.xacro" />
   <xacro:include filename="$(find cob_hardware_config)/robots/raw3-5/urdf/properties.urdf.xacro" />
+  <xacro:include filename="$(find sick_visionary_t_driver)/description/urdf/visionary_t_macro.urdf.xacro" />
   <!-- raw base -->
   <xacro:include filename="$(find raw_description)/urdf/base_short/base.urdf.xacro" />
@@ -15,3 +16,7 @@
     <origin xyz="-0.348 0  0.96" rpy="0 0 0" />
   </xacro:ati_mini58>
+  <xacro:sick_visionary_t parent="base_link" has_holder="true" holder_tilt="${-25/180*pi}">
+    <origin xyz="0.0 0.0 0.0" rpy="${pi} 0 0" />
+  </xacro:sick_visionary_t>
+
 </robot>
