Commit message: Added additional files

File: urdf/sr2.urdf.xacro (robot description, xacro)
@@ -4,5 +4,5 @@
   <xacro:arg name="neck" default="false"/>
   <xacro:arg name="fts" default="false"/>
-  <xacro:arg name="real_fts" default="false"/>
+  <xacro:arg name="fts_sim" default="false"/>
   <xacro:arg name="sick_visionary_t" default="false"/>
   <!-- common stuff -->
@@ -13,12 +13,22 @@
   <!-- raw base -->
   <xacro:include filename="$(find raw_description)/urdf/base_short/base.urdf.xacro" />
+  <!-- sensors -->
+  <xacro:include filename="$(find cob_description)/urdf/sensors/sick_s300_laser.urdf.xacro"/>
   <!-- composition of the robot -->
   <xacro:raw_base name="base"/>
+  <!-- base laser front -->
+  <xacro:sick_s300_laser_v0 name="base_laser_front" parent="base">
+    <origin xyz="${laser_front_x} ${laser_front_y} ${laser_front_z}" rpy="${laser_front_roll} ${laser_front_pitch} ${laser_front_yaw}" />
+  </xacro:sick_s300_laser_v0>
+  <!-- base laser rear -->
+  <xacro:sick_s300_laser_v0 name="base_laser_rear" parent="base">
+    <origin xyz="${laser_rear_x} ${laser_rear_y} ${laser_rear_z}" rpy="${laser_rear_roll} ${laser_rear_pitch} ${laser_rear_yaw}" />
+  </xacro:sick_s300_laser_v0>
   <!-- COMPONENTS -->
   <joint name="led_rectangle_joint" type="fixed">
-            <origin xyz="0 0 0" rpy="0 0 0" />
-            <parent link="base_link"/>
-            <child link="led_rectangle_link" />
-        </joint>
+    <origin xyz="0 0 0" rpy="0 0 0" />
+    <parent link="base_link"/>
+    <child link="led_rectangle_link" />
+  </joint>
   <link name="led_rectangle_link">
   </link>

Commit message: Added frames for robotrainer markers

File: urdf/sr2.urdf.xacro (robot description, xacro)
@@ -26,4 +26,26 @@
     <origin xyz="${laser_rear_x} ${laser_rear_y} ${laser_rear_z}" rpy="${laser_rear_roll} ${laser_rear_pitch} ${laser_rear_yaw}" />
   </xacro:sick_s300_laser_v0>
+  <!-- RoboTrainer Joints -->
+  <joint name="robotrainer_front_marker_joint" type="fixed">
+    <origin xyz="0.4 0 0" rpy="0 0 0" />
+    <parent link="base_link"/>
+    <child link="robotrainer_front_marker" />
+  </joint>
+  <link name="robotrainer_front_marker">
+  </link>
+  <joint name="robotrainer_left_marker_joint" type="fixed">
+    <origin xyz="0 0.2 0" rpy="0 0 0" />
+    <parent link="base_link"/>
+    <child link="robotrainer_left_marker" />
+  </joint>
+  <link name="robotrainer_left_marker">
+  </link>
+  <joint name="robotrainer_right_marker_joint" type="fixed">
+    <origin xyz="0 0.2 0" rpy="0 0 0" />
+    <parent link="base_link"/>
+    <child link="robotrainer_right_marker" />
+  </joint>
+  <link name="robotrainer_right_marker">
+  </link>
   <!-- COMPONENTS -->
   <joint name="led_rectangle_joint" type="fixed">

Commit message: Added rotations of markers on the platform

File: urdf/sr2.urdf.xacro (robot description, xacro)
@@ -28,5 +28,5 @@
   <!-- RoboTrainer Joints -->
   <joint name="robotrainer_front_marker_joint" type="fixed">
-    <origin xyz="0.4 0 0" rpy="0 0 0" />
+    <origin xyz="0.375 0 0.3" rpy="0 0 0" />
     <parent link="base_link"/>
     <child link="robotrainer_front_marker" />
@@ -35,5 +35,5 @@
   </link>
   <joint name="robotrainer_left_marker_joint" type="fixed">
-    <origin xyz="0 0.2 0" rpy="0 0 0" />
+    <origin xyz="0 0.28 0.3" rpy="0 0 0" />
     <parent link="base_link"/>
     <child link="robotrainer_left_marker" />
@@ -42,5 +42,5 @@
   </link>
   <joint name="robotrainer_right_marker_joint" type="fixed">
-    <origin xyz="0 0.2 0" rpy="0 0 0" />
+    <origin xyz="0 -0.28 0.3" rpy="0 0 ${pi}" />
     <parent link="base_link"/>
     <child link="robotrainer_right_marker" />
