Commit message: tested on sr2: simulation to do

File: urdf/components/fts.urdf.xacro (robot description, xacro)
@@ -2,12 +2,12 @@
 <robot xmlns:xacro="http://www.ros.org/wiki/xacro" name="sr2_fts" >
   <!--<xacro:arg name="real_fts" default="false"/>-->
-  <xacro:if value="${sim}">
+  <xacro:if value="$(arg sim)">
     <xacro:include filename="$(find ati_force_torque)/description/urdf/macros/mini58_sim.urdf.xacro" />
   </xacro:if>
-  <xacro:unless value="${sim}">
-    <xacro:include filename="$(find ati_force_torque)/description/urdf/macros/mini58_sim.urdf.xacro" />
+  <xacro:unless value="$(arg sim)">
+    <xacro:include filename="$(find ati_force_torque)/description/urdf/macros/mini58.urdf.xacro" />
   </xacro:unless>
-  <xacro:ati_mini58 name="fts" parent="base_link">
+<!--  <xacro:ati_mini58 name="fts" parent="base_link">
     <origin xyz="-0.348 0  0.96" rpy="0 0 0" />
-  </xacro:ati_mini58>
+  </xacro:ati_mini58>-->
 </robot>

File: urdf/sr2.urdf.xacro (robot description, xacro)
@@ -16,5 +16,5 @@
   <xacro:raw_base name="base"/>
   <!-- COMPONENTS -->
-  <joint name="${name}_reference_joint" type="fixed">
+  <joint name="led_rectangle_joint" type="fixed">
             <origin xyz="0 0 0" rpy="0 0 0" />
             <parent link="base_link"/>
@@ -23,11 +23,11 @@
   <link name="led_rectangle_link">
   </link>
-  <xacro:if value="${neck}">
+  <xacro:if value="$(arg neck)">
     <xacro:include filename="$(find sr2_bringup)/urdf/components/neck.urdf.xacro" />
   </xacro:if>
-  <xacro:if value="${fts}">
+  <xacro:if value="$(arg fts)">
     <xacro:include filename="$(find sr2_bringup)/urdf/components/fts.urdf.xacro" />
   </xacro:if>
-  <xacro:if value="${sick_visionary_t}">
+  <xacro:if value="$(arg sick_visionary_t)">
     <xacro:include filename="$(find sr2_bringup)/urdf/components/sick_visionary_t.urdf.xacro" />
   </xacro:if>
