Commit message: Today was working to start the robot and robotrainer (robot with FTS)

File: urdf/components/neck.urdf.xacro (robot description, xacro)
@@ -2,8 +2,10 @@
 <robot xmlns:xacro="http://www.ros.org/wiki/xacro" name="sr2_neck" >
   <!-- common stuff -->
-  <xacro:include filename="$(find schunk_description)/urdf/common.xacro" />
+<!--  <xacro:include filename="$(find schunk_description)/urdf/common.xacro" />
   <xacro:include filename="$(find schunk_description)/urdf/materials.urdf.xacro" />
+-->
   <!-- schunk powercube -->
   <xacro:include filename="$(find schunk_description)/urdf/pw70/pw70.urdf.xacro" />
+  <!--<link name="base_link" /> -->
   <xacro:schunk_pw70 name="neck" parent="base_link" is_upsidedown="true">
     <origin xyz="0 -0.24 0.836" rpy="0 0 ${-1/2 * M_PI}" />

Commit message: Added object_tracking_robot.launch

File: urdf/components/neck.urdf.xacro (robot description, xacro)
@@ -9,5 +9,5 @@
   <!--<link name="base_link" /> -->
   <xacro:schunk_pw70 name="neck" parent="base_link" is_upsidedown="true">
-    <origin xyz="0 -0.24 0.836" rpy="0 0 ${-1/2 * M_PI}" />
+    <origin xyz="0 -0.24 0.836" rpy="0 0 ${pi}" />
   </xacro:schunk_pw70>
 </robot>

File: urdf/components/object_tracking.urdf.xacro (robot description, xacro)
@@ -1,16 +1,14 @@
 <?xml version="1.0"?>
 <robot xmlns:xacro="http://www.ros.org/wiki/xacro" name="sr2_object_tracking" >
-    <joint name="base_map" type="fixed">
+<!--    <joint name="base_map" type="fixed">
             <origin xyz="0 0 0" rpy="0 0 0" />
             <parent link="base_link"/>
             <child link="map" />
-        </joint>
-    <link name="map">
-    </link>
+    </joint>-->
     <joint name="map_conveyor" type="fixed">
-            <origin xyz="0 0 60" rpy="0 0 0" />
-            <parent link="map"/>
-            <child link="conveyor" />
-        </joint>
+        <origin xyz="0 0 60" rpy="0 0 0" />
+        <parent link="base_footprint"/>
+        <child link="conveyor" />
+    </joint>
     <link name="conveyor">
     </link>
