Commit message: Uncommited changes; Change can device; Fix transform with PI

File: urdf/components/mini58.urdf.xacro (robot description, xacro)
@@ -34,5 +34,5 @@
 -->
         <joint name="${name}_reference_joint" type="fixed">
-            <origin xyz="0 0 0" rpy="0 0 -2.22068070" />
+            <origin xyz="0 0 0" rpy="0 0 ${M_PI*(-120)/180}" />
             <parent link="${name}_base_link"/>
             <child link="${name}_reference_link" />
